File: kicad/V1.0.1.sch (KiCad schematic (older format))
At the start: 20 parts, among them IC1 OPA2134P, U1 TLE2426CP

Commit message: Modified slightly to fix some ERC issues
Parts:
- 9V9: footprint BATTERY_AB9V -> V1.0.1:BATTERY_AB9V
- C1: footprint RCL_E3_5-8 -> V1.0.1:RCL_E3_5-8
- C1V+9, C1V-9: footprint CAPACITOR-WIMA_C2.5-2 -> V1.0.1:CAPACITOR-WIMA_C2.5-2
- C2L9, C2R9: footprint CAPACITOR-WIMA_C5B5 -> V1.0.1:CAPACITOR-WIMA_C5B5
- C4: footprint CAPACITOR-WIMA_C5B2.5 -> V1.0.1:CAPACITOR-WIMA_C5B2.5
- IC1: footprint AKAFUGU_DIL-8 -> V1.0.1:AKAFUGU_DIL-8
- JACK-IN9, JACK-OUT9: footprint AKAFUGU_STX3100 -> V1.0.1:AKAFUGU_STX3100
- R3L9, R3R9, R4L9, R4R9, R5L9, R5R9, R6L9, R6R9: footprint RESISTOR_0207_2V -> V1.0.1:RESISTOR_0207_2V
- U$1: footprint AUDIO-POTS_ALPS_RK0971221Z0X -> V1.0.1:AUDIO-POTS_ALPS_RK0971221Z0X
- U1: footprint TLE2426_DIP-8 -> V1.0.1:TLE2426_DIP-8
Changed lines of the file:
@@
 EESchema Schematic File Version 2
 LIBS:V1.0.1
-EELAYER 27 0
+LIBS:V1.0.1-cache
+EELAYER 25 0
 EELAYER END
 $Descr A4 11693 8268
@@
 F 0 "9V9" H 7725 5675 70  0000 L BNN
 F 1 "AB9V" H 7725 5350 70  0000 L BNN
-F 2 "BATTERY_AB9V" H 7725 5350 70  0001 L BNN
+F 2 "V1.0.1:BATTERY_AB9V" H 7725 5350 70  0001 L BNN
 F 3 "" H 7950 5550 60  0001 C CNN
 	1    7950 5550
@@
 F 0 "C1" H 8890 5474 70  0000 L BNN
 F 1 "220uF" H 8889 5285 70  0000 L BNN
-F 2 "RCL_E3_5-8" H 8840 5240 65  0001 L TNN
+F 2 "V1.0.1:RCL_E3_5-8" H 8840 5240 65  0001 L TNN
 F 3 "" H 8850 5450 60  0001 C CNN
 	1    8850 5450
@@
 F 0 "C1V+9" H 10110 5265 70  0000 L BNN
 F 1 "0.068uF" H 10110 5065 70  0000 L BNN
-F 2 "CAPACITOR-WIMA_C2.5-2" H 10040 5040 65  0001 L TNN
+F 2 "V1.0.1:CAPACITOR-WIMA_C2.5-2" H 10040 5040 65  0001 L TNN
 F 3 "" H 10050 5250 60  0001 C CNN
 	1    10050 5250
@@
 F 0 "C1V-9" H 10110 5765 70  0000 L BNN
 F 1 "0.068uF" H 10110 5565 70  0000 L BNN
-F 2 "CAPACITOR-WIMA_C2.5-2" H 10040 5540 65  0001 L TNN
+F 2 "V1.0.1:CAPACITOR-WIMA_C2.5-2" H 10040 5540 65  0001 L TNN
 F 3 "" H 10050 5750 60  0001 C CNN
 	1    10050 5750
@@
 F 0 "C2L9" H 4360 2065 70  0000 L BNN
 F 1 "0.1uF" H 4360 1865 70  0000 L BNN
-F 2 "CAPACITOR-WIMA_C5B5" H 4290 1840 65  0001 L TNN
+F 2 "V1.0.1:CAPACITOR-WIMA_C5B5" H 4290 1840 65  0001 L TNN
 F 3 "" H 4300 2050 60  0001 C CNN
 	1    4300 2050
@@
 F 0 "C2R9" H 3560 5265 70  0000 L BNN
 F 1 "0.1uF" H 3560 5065 70  0000 L BNN
-F 2 "CAPACITOR-WIMA_C5B5" H 3490 5040 65  0001 L TNN
+F 2 "V1.0.1:CAPACITOR-WIMA_C5B5" H 3490 5040 65  0001 L TNN
 F 3 "" H 3500 5250 60  0001 C CNN
 	1    3500 5250
@@
 F 0 "C4" H 9710 5864 70  0000 L BNN
 F 1 "1uF" H 9709 5665 70  0000 L BNN
-F 2 "CAPACITOR-WIMA_C5B2.5" H 9640 5640 65  0001 L TNN
+F 2 "V1.0.1:CAPACITOR-WIMA_C5B2.5" H 9640 5640 65  0001 L TNN
 F 3 "" H 9650 5850 60  0001 C CNN
 	1    9650 5850
@@
 F 0 "IC1" H 4700 5575 70  0000 L BNN
 F 1 "OPA2134P" H 4699 5150 70  0000 L BNN
-F 2 "AKAFUGU_DIL-8" H 4590 5140 65  0001 L TNN
+F 2 "V1.0.1:AKAFUGU_DIL-8" H 4590 5140 65  0001 L TNN
 F 3 "" H 4600 5350 60  0001 C CNN
 	1    4600 5350
@@
 F 0 "IC1" H 3300 2375 70  0000 L BNN
 F 1 "OPA2134P" H 3299 1950 70  0000 L BNN
-F 2 "AKAFUGU_DIL-8" H 3190 1940 65  0001 L TNN
+F 2 "V1.0.1:AKAFUGU_DIL-8" H 3190 1940 65  0001 L TNN
 F 3 "" H 3200 2150 60  0001 C CNN
 	2    3200 2150
@@
 F 0 "JACK-IN9" H 5400 3200 70  0000 L BNN
 F 1 "STEREOJACK" H 5400 2650 70  0000 L BNN
-F 2 "AKAFUGU_STX3100" H 5690 2840 65  0001 L TNN
+F 2 "V1.0.1:AKAFUGU_STX3100" H 5690 2840 65  0001 L TNN
 F 3 "" H 5700 3050 60  0001 C CNN
 	1    5700 3050
@@
 F 0 "JACK-OUT9" H 5400 4100 70  0000 L BNN
 F 1 "STEREOJACK" H 5400 3550 70  0000 L BNN
-F 2 "AKAFUGU_STX3100" H 5690 3740 65  0001 L TNN
+F 2 "V1.0.1:AKAFUGU_STX3100" H 5690 3740 65  0001 L TNN
 F 3 "" H 5700 3950 60  0001 C CNN
 	1    5700 3950
@@
 F 0 "R3L9" H 3750 2409 70  0000 L BNN
 F 1 "100k" H 3750 2220 70  0000 L BNN
-F 2 "RESISTOR_0207_2V" H 3890 2140 65  0001 L TNN
+F 2 "V1.0.1:RESISTOR_0207_2V" H 3890 2140 65  0001 L TNN
 F 3 "" H 3900 2350 60  0001 C CNN
 	1    3900 2350
@@
 F 0 "R3R9" H 3750 5609 70  0000 L BNN
 F 1 "100k" H 3750 5420 70  0000 L BNN
-F 2 "RESISTOR_0207_2V" H 3890 5340 65  0001 L TNN
+F 2 "V1.0.1:RESISTOR_0207_2V" H 3890 5340 65  0001 L TNN
 F 3 "" H 3900 5550 60  0001 C CNN
 	1    3900 5550
@@
 F 0 "R4L9" H 3450 3209 70  0000 L BNN
 F 1 "2k" H 3450 3020 70  0000 L BNN
-F 2 "RESISTOR_0207_2V" H 3590 2940 65  0001 L TNN
+F 2 "V1.0.1:RESISTOR_0207_2V" H 3590 2940 65  0001 L TNN
 F 3 "" H 3600 3150 60  0001 C CNN
 	1    3600 3150
@@
 F 0 "R4R9" H 4050 6409 70  0000 L BNN
 F 1 "2k" H 4050 6220 70  0000 L BNN
-F 2 "RESISTOR_0207_2V" H 4190 6140 65  0001 L TNN
+F 2 "V1.0.1:RESISTOR_0207_2V" H 4190 6140 65  0001 L TNN
 F 3 "" H 4200 6350 60  0001 C CNN
 	1    4200 6350
@@
 F 0 "R5L9" H 2450 2208 70  0000 L BNN
 F 1 "47R" H 2450 2020 70  0000 L BNN
-F 2 "RESISTOR_0207_2V" H 2590 1940 65  0001 L TNN
+F 2 "V1.0.1:RESISTOR_0207_2V" H 2590 1940 65  0001 L TNN
 F 3 "" H 2600 2150 60  0001 C CNN
 	1    2600 2150
@@
 F 0 "R5R9" H 5050 5408 70  0000 L BNN
 F 1 "47R" H 5050 5220 70  0000 L BNN
-F 2 "RESISTOR_0207_2V" H 5190 5140 65  0001 L TNN
+F 2 "V1.0.1:RESISTOR_0207_2V" H 5190 5140 65  0001 L TNN
 F 3 "" H 5200 5350 60  0001 C CNN
 	1    5200 5350
@@
 F 0 "R6L9" H 2750 2908 70  0000 L BNN
 F 1 "10k" H 2750 2720 70  0000 L BNN
-F 2 "RESISTOR_0207_2V" H 2890 2640 65  0001 L TNN
+F 2 "V1.0.1:RESISTOR_0207_2V" H 2890 2640 65  0001 L TNN
 F 3 "" H 2900 2850 60  0001 C CNN
 	1    2900 2850
@@
 F 0 "R6R9" H 4750 6108 70  0000 L BNN
 F 1 "10k" H 4750 5920 70  0000 L BNN
-F 2 "RESISTOR_0207_2V" H 4890 5840 65  0001 L TNN
+F 2 "V1.0.1:RESISTOR_0207_2V" H 4890 5840 65  0001 L TNN
 F 3 "" H 4900 6050 60  0001 C CNN
 	1    4900 6050
@@
 F 0 "U$1" H 8440 5040 65  0001 L TNN
 F 1 "~" H 8440 4940 65  0001 L TNN
-F 2 "AUDIO-POTS_ALPS_RK0971221Z0X" H 8440 4840 65  0001 L TNN
+F 2 "V1.0.1:AUDIO-POTS_ALPS_RK0971221Z0X" H 8440 4840 65  0001 L TNN
 F 3 "" H 8450 5050 60  0001 C CNN
 	1    8450 5050
@@
 F 0 "U$1" V 4800 1951 70  0000 L BNN
 F 1 "~" H 4990 1940 65  0001 L TNN
-F 2 "AUDIO-POTS_ALPS_RK0971221Z0X" H 4990 1840 65  0001 L TNN
+F 2 "V1.0.1:AUDIO-POTS_ALPS_RK0971221Z0X" H 4990 1840 65  0001 L TNN
 F 3 "" H 5000 2050 60  0001 C CNN
 	2    5000 2050
@@
 F 0 "U$1" V 2600 5151 70  0000 L BNN
 F 1 "~" H 2790 5140 65  0001 L TNN
-F 2 "AUDIO-POTS_ALPS_RK0971221Z0X" H 2790 5040 65  0001 L TNN
+F 2 "V1.0.1:AUDIO-POTS_ALPS_RK0971221Z0X" H 2790 5040 65  0001 L TNN
 F 3 "" H 2800 5250 60  0001 C CNN
 	3    2800 5250
@@
 F 0 "U1" H 9450 5775 70  0000 L BNN
 F 1 "TLE2426CP" H 9450 5650 70  0000 L BNN
-F 2 "TLE2426_DIP-8" H 9340 5340 65  0001 L TNN
+F 2 "V1.0.1:TLE2426_DIP-8" H 9340 5340 65  0001 L TNN
 F 3 "" H 9350 5550 60  0001 C CNN
 	1    9350 5550
@@
 	1800 2150 2400 2150
 Wire Wire Line
-	2300 2150 2300 2850
+	2300 2850 2300 2150
 Connection ~ 2300 2150
 Text Label 2200 2150 2    65   ~ 0
@@
 	5400 5350 6000 5350
 Wire Wire Line
-	5500 5350 5500 6050
+	5500 6050 5500 5350
 Connection ~ 5500 5350
 Text Label 5600 5350 0    65   ~ 0
@@
 Text Label 3300 5250 2    10   ~ 0
 VOLUME-OUT-R
-Entry Wire Line
-	7350 3950 7450 4050
 $EndSCHEMATC
